File: Spojko_Hardware/Spojko/SpojkoKonektori.sch (KiCad schematic (older format))
At the start: 14 parts, among them J3 CONN_02X40, J4 CONN_02X40, J5 CONN_02X40, J6 CONN_02X40, J7 CONN_02X40, J8 CONN_02X40

Commit message: Popravljena greska u konektorima
Connections:
- net at J3.27 (P27), J3.28 (P28), J4.27 (P27)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: now also J7.27 (P27), J7.28 (P28), J8.27 (P27), J8.28 (P28)
- net at J3.29 (P29), J3.30 (P30), J4.29 (P29)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: now also J7.29 (P29), J7.30 (P30), J8.29 (P29), J8.30 (P30)
- net at J3.31 (P31), J3.32 (P32), J4.31 (P31)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: now also J7.31 (P31), J7.32 (P32), J8.31 (P31), J8.32 (P32)
- net at J3.33 (P33), J3.34 (P34), J4.33 (P33)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: now also J7.33 (P33), J7.34 (P34), J8.33 (P33), J8.34 (P34)
- net at J3.35 (P35), J3.36 (P36), J4.35 (P35)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: now also J7.35 (P35), J7.36 (P36), J8.35 (P35), J8.36 (P36)
- net at J3.37 (P37), J3.38 (P38), J4.37 (P37)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: now also J7.37 (P37), J7.38 (P38), J8.37 (P37), J8.38 (P38)
- net at J3.39 (P39), J3.40 (P40), J4.39 (P39)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: now also J7.39 (P39)
- net at J3.41 (P41), J3.42 (P42), J4.41 (P41)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: now also J7.41 (P41), J7.42 (P42), J8.41 (P41), J8.42 (P42)
- net at J7.40 (P40), J8.39 (P39), J8.40 (P40): no longer J7.39 (P39)
Changed lines of the file:
@@
 EESchema Schematic File Version 2
+LIBS:Spojko-cache
 LIBS:power
 LIBS:device
@@
 LIBS:contrib
 LIBS:valves
-LIBS:cat24c32hu4i-gt3
-LIBS:DMMT5401
-LIBS:fdc5614p
-LIBS:lm1117
-LIBS:lm3489
-LIBS:max1164x
-LIBS:mcp23017
-LIBS:raspberry_pi_+_conn
 LIBS:Symbols_DCDC-ACDC-Converter_RevC_20Jul2012
 LIBS:Symbols_EN60617_13Mar2013
@@
 LIBS:Symbols_Transformer-Diskrete_RevA
 LIBS:SymbolsSimilarEN60617+oldDIN617-RevE8
-LIBS:vLM2596
-LIBS:ESP8266
-LIBS:vESP-12e
-LIBS:vPower5V-3V3
 LIBS:switches
 LIBS:sensors
-LIBS:sefrtsrts
-LIBS:Spojko-cache
 EELAYER 25 0
 EELAYER END
 $Descr A4 11693 8268
 encoding utf-8
-Sheet 6 5
+Sheet 5 5
 Title ""
 Date ""
@@
 	1500 2900 1700 2900
 Wire Wire Line
-	1250 3000 7000 3000
-Wire Wire Line
-	7050 3000 10650 3000
-Wire Wire Line
-	1250 3100 7000 3100
-Wire Wire Line
-	7050 3100 10650 3100
-Wire Wire Line
-	1250 3200 7000 3200
-Wire Wire Line
-	7050 3200 10650 3200
-Wire Wire Line
-	1250 3300 7000 3300
-Wire Wire Line
-	7050 3300 10650 3300
-Wire Wire Line
-	1250 3400 7000 3400
-Wire Wire Line
-	7050 3400 10650 3400
-Wire Wire Line
-	1250 3500 7000 3500
-Wire Wire Line
-	7050 3500 10650 3500
-Wire Wire Line
-	1250 3600 7000 3600
-Wire Wire Line
-	7050 3600 10650 3600
-Wire Wire Line
-	1250 3700 7000 3700
-Wire Wire Line
-	7050 3700 10650 3700
+	1250 3000 10650 3000
+Wire Wire Line
+	1250 3100 10650 3100
+Wire Wire Line
+	1250 3200 10650 3200
+Wire Wire Line
+	1250 3300 10650 3300
+Wire Wire Line
+	1250 3400 10650 3400
+Wire Wire Line
+	1250 3500 10650 3500
+Wire Wire Line
+	1250 3600 8150 3600
+Wire Wire Line
+	1250 3700 10650 3700
 Wire Wire Line
 	2200 1800 2400 1800
@@
 	8650 1700 8850 1700
 Connection ~ 10150 3000
+Connection ~ 10150 3100
+Connection ~ 10150 3200
+Connection ~ 10150 3300
+Connection ~ 10150 3400
+Connection ~ 10150 3500
+Connection ~ 10150 3600
+Connection ~ 10150 3700
+Connection ~ 7000 3000
+Connection ~ 7000 3100
+Connection ~ 7000 3200
+Connection ~ 7000 3300
+Connection ~ 7000 3400
+Connection ~ 7000 3500
+Connection ~ 7000 3600
+Connection ~ 7000 3700
+Wire Wire Line
+	8200 3600 10650 3600
 Connection ~ 8650 3000
-Connection ~ 10150 3100
 Connection ~ 8650 3100
-Connection ~ 10150 3200
 Connection ~ 8650 3200
-Connection ~ 10150 3300
 Connection ~ 8650 3300
-Connection ~ 10150 3400
 Connection ~ 8650 3400
-Connection ~ 10150 3500
 Connection ~ 8650 3500
-Connection ~ 10150 3600
 Connection ~ 8650 3600
-Connection ~ 10150 3700
 Connection ~ 8650 3700
 $EndSCHEMATC
