File: Spojko_Hardware/Spojko/Spojko.sch (KiCad schematic (older format))
At the start: 25 parts, among them J1 CONN_01X02, J2 CONN_01X06, P1 Raspberry_Pi, Q1 BSS138, Q2 BSS138, SW1 SW_Reset, SW2 SW_Flash, U1 ESP-12E, U6 DHT11

Commit message: Spojko zavrsen, valjda
Connections:
- net RST: now reaches P1.26 (GPIO7/SPI_CE1)
Changed lines of the file:
@@
 Wire Wire Line
 	10600 5100 10600 5900
+Text GLabel 5150 4200 2    60   Input ~ 0
+RST
+Wire Wire Line
+	5150 4200 5000 4200
 $EndSCHEMATC
