File: Spojko_Hardware/Spojko/Spojko.sch (KiCad schematic (older format))
At the start: 25 parts, among them J1 CONN_01X02, J2 CONN_01X06, P1 Raspberry_Pi, Q1 BSS138, Q2 BSS138, SW1 SW_Reset, SW2 SW_Flash, U1 ESP-12E, U6 DHT11

Commit message: Pre Develope
Connections:
- net RST: now also P1.29 (GPIO5); no longer P1.26 (GPIO7/SPI_CE1)
- net GPIO17: now reaches P1.11 (GPIO17)
- net GPIO27: now reaches P1.13 (GPIO27)
- net GPIO22: now reaches P1.15 (GPIO22)
- net GPIO10-SPI-MOSI: now reaches P1.19 (GPIO10/SPI_M0SI)
- net GPIO09-SPI-MISO: now reaches P1.21 (GPIO9/SPI_MISO)
- net GPI11-SPI-SCLK: now reaches P1.23 (GPIO11/SPI_SCLK)
- net GPIO8-SPIO-CE0: now reaches P1.24 (GPIO8/SPI_CE0)
- net GPIO13: now reaches P1.33 (GPIO13)
- net GPIO4: now reaches P1.7 (GPIO4/GPCLK0)
- new net GPIO7-SPI-CE1: P1.26 (GPIO7/SPI_CE1)
Changed lines of the file:
@@
 Wire Wire Line
 	10600 5100 10600 5900
-Text GLabel 4850 4100 2    60   Input ~ 0
+Text GLabel 4850 4600 2    60   Input ~ 0
 RST
-Wire Wire Line
-	4850 4100 4700 4100
 Wire Wire Line
 	2050 3850 2050 3950
@@
 Wire Wire Line
 	3750 1650 3400 1650
+Text GLabel 4850 4500 2    60   Input ~ 0
+GPIO4
+Text GLabel 4850 4900 2    60   Input ~ 0
+GPIO13
+Text GLabel 4850 5100 2    60   Input ~ 0
+GPIO17
+Text GLabel 4850 5600 2    60   Input ~ 0
+GPIO22
+Text GLabel 4850 6100 2    60   Input ~ 0
+GPIO27
+Wire Wire Line
+	4700 6100 4850 6100
+Wire Wire Line
+	4700 5600 4850 5600
+Wire Wire Line
+	4700 5100 4850 5100
+Wire Wire Line
+	4700 4900 4850 4900
+Wire Wire Line
+	4700 4700 4850 4700
+Wire Wire Line
+	4700 4600 4850 4600
+Wire Wire Line
+	4700 4500 4850 4500
+Text GLabel 4850 3700 2    60   Input ~ 0
+GPIO10-SPI-MOSI
+Text GLabel 4850 3800 2    60   Input ~ 0
+GPIO09-SPI-MISO
+Text GLabel 4850 3900 2    60   Input ~ 0
+GPI11-SPI-SCLK
+Text GLabel 4850 4000 2    60   Input ~ 0
+GPIO8-SPIO-CE0
+Wire Wire Line
+	4700 3700 4850 3700
+Wire Wire Line
+	4700 3800 4850 3800
+Wire Wire Line
+	4700 3900 4850 3900
+Wire Wire Line
+	4700 4000 4850 4000
+Text GLabel 4850 4100 2    60   Input ~ 0
+GPIO7-SPI-CE1
+Wire Wire Line
+	4850 4100 4700 4100
 $EndSCHEMATC
