File: Spojko_Hardware/Spojko/Spojko.kicad_pcb (KiCad board)
At the start: 2 copper layers, 254 x 139.7 mm, 42 parts, among them J1 CONN_01X02, J2 CONN_01X06, J3 CONN_02X40, J4 CONN_02X40, J5 CONN_02X40, J6 CONN_02X40, J7 CONN_02X40, J8 CONN_02X40, P1 Raspberry_Pi, Q1 BSS138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

Commit message: FirstCommit
Routing:
- net TXD: track 0.00 -> 227.5 mm, vias 0 -> 6
- net RXD: track 0.00 -> 227.1 mm, vias 0 -> 4
- net SCL: track 0.00 -> 222.1 mm
- net SDA: track 0.00 -> 217.2 mm
- net SDA1: track 0.00 -> 144.1 mm
- net SCL1: track 0.00 -> 139.4 mm, vias 0 -> 1
- net RST: track 0.00 -> 116.8 mm
- net +3V3: track 0.00 -> 111.7 mm, vias 0 -> 1
- net GPIO20: track 0.00 -> 109.5 mm, vias 0 -> 2
- net GPIO21: track 0.00 -> 107.0 mm
- net GPIO16: track 0.00 -> 98.8 mm
- net Net-(J3-Pad41): track 0.00 -> 98.4 mm
- net Net-(J3-Pad39): track 0.00 -> 98.1 mm
- net Net-(J3-Pad37): track 0.00 -> 97.4 mm
- net Net-(J3-Pad35): track 0.00 -> 97.0 mm
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- added copper zone on B.Cu, net +24V
- added copper zone on B.Cu, net +3V3
- added copper zone on B.Cu, net +5V
- added copper zone on F.Cu, net GND
- added copper zone on F.Cu, net GND24V

Commit message: Spojko zavrsen, valjda
Parts:
- moved SW2 2.84 mm to (109.2, 124.5)
- moved C2 2.81 mm to (91.7, 107.7)
- moved C3 2.54 mm to (96.5, 108.0)
Connections:
- J7 pad 27: Net-(J7-Pad27) -> Net-(J3-Pad27)
- J7 pad 28: Net-(J7-Pad27) -> Net-(J3-Pad27)
- J7 pad 29: Net-(J7-Pad29) -> Net-(J3-Pad29)
- J7 pad 30: Net-(J7-Pad29) -> Net-(J3-Pad29)
- J7 pad 31: Net-(J7-Pad31) -> Net-(J3-Pad31)
- J7 pad 32: Net-(J7-Pad31) -> Net-(J3-Pad31)
- J7 pad 33: Net-(J7-Pad33) -> Net-(J3-Pad33)
- J7 pad 34: Net-(J7-Pad33) -> Net-(J3-Pad33)
- J7 pad 35: Net-(J7-Pad35) -> Net-(J3-Pad35)
- J7 pad 36: Net-(J7-Pad35) -> Net-(J3-Pad35)
- J7 pad 37: Net-(J7-Pad37) -> Net-(J3-Pad37)
- J7 pad 38: Net-(J7-Pad37) -> Net-(J3-Pad37)
- J7 pad 39: Net-(J7-Pad39) -> Net-(J3-Pad39)
- J7 pad 40: Net-(J7-Pad39) -> Net-(J7-Pad40)
- J7 pad 41: Net-(J7-Pad41) -> Net-(J3-Pad41)
- J7 pad 42: Net-(J7-Pad41) -> Net-(J3-Pad41)
- J8 pad 27: Net-(J7-Pad27) -> Net-(J3-Pad27)
- J8 pad 28: Net-(J7-Pad27) -> Net-(J3-Pad27)
- J8 pad 29: Net-(J7-Pad29) -> Net-(J3-Pad29)
- J8 pad 30: Net-(J7-Pad29) -> Net-(J3-Pad29)
- J8 pad 31: Net-(J7-Pad31) -> Net-(J3-Pad31)
- J8 pad 32: Net-(J7-Pad31) -> Net-(J3-Pad31)
- J8 pad 33: Net-(J7-Pad33) -> Net-(J3-Pad33)
- J8 pad 34: Net-(J7-Pad33) -> Net-(J3-Pad33)
- J8 pad 35: Net-(J7-Pad35) -> Net-(J3-Pad35)
- J8 pad 36: Net-(J7-Pad35) -> Net-(J3-Pad35)
- J8 pad 37: Net-(J7-Pad37) -> Net-(J3-Pad37)
- J8 pad 38: Net-(J7-Pad37) -> Net-(J3-Pad37)
- J8 pad 39: Net-(J7-Pad39) -> Net-(J7-Pad40)
- J8 pad 40: Net-(J7-Pad39) -> Net-(J7-Pad40)
- J8 pad 41: Net-(J7-Pad41) -> Net-(J3-Pad41)
- J8 pad 42: Net-(J7-Pad41) -> Net-(J3-Pad41)
- P1 pad 26: Net-(P1-Pad26) -> RST
Routing:
- net RST: track 116.8 -> 225.4 mm, vias 0 -> 4
- net Net-(J3-Pad41): track 98.4 -> 136.5 mm
- net Net-(J3-Pad37): track 97.4 -> 135.5 mm
- net Net-(J3-Pad33): track 96.3 -> 134.4 mm
- net Net-(J3-Pad29): track 95.2 -> 133.4 mm
- net Net-(J3-Pad27): track 95.8 -> 133.9 mm
- net Net-(J3-Pad35): track 97.0 -> 134.9 mm
- net Net-(J3-Pad31): track 96.0 -> 133.9 mm
- net Net-(J3-Pad39): track 98.1 -> 123.6 mm
- net GND: track 29.9 -> 8.55 mm, vias 4 -> 2
- net GPIO20: track 109.5 -> 127.3 mm
- net Net-(J7-Pad41): track 15.2 -> 0.00 mm
- net Net-(J7-Pad39): track 15.2 -> 0.00 mm
- net Net-(J7-Pad37): track 15.2 -> 0.00 mm
- net Net-(J7-Pad35): track 15.2 -> 0.00 mm
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
Commit message: Izmene predlozi matori
Other:
- net class +5V: clearance 0.3 -> 0.6
Changed lines of the file:
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@@
   )
   (net_class +5V ""
-    (clearance 0.3)
+    (clearance 0.6)
     (trace_width 0.781437)
     (via_dia 0.6)
@@
     (pad 80 thru_hole oval (at 2.54 99.06) (size 1.7 1.7) (drill 1) (layers *.Cu *.Mask)
       (net 12 SCL))
-    (model ${KISYS3DMOD}/Pin_Headers.3dshapes/Pin_Header_Straight_2x40_Pitch2.54mm.wrl
-      (at (xyz 0 0 0))
-      (scale (xyz 1 1 1))
-      (rotate (xyz 0 0 0))
-    )
   )
   (module project_footprints:ESP-12E (layer F.Cu)
@@
     (pad 80 thru_hole oval (at 2.54 99.06) (size 1.7 1.7) (drill 1) (layers *.Cu *.Mask)
       (net 12 SCL))
-    (model ${KISYS3DMOD}/Pin_Headers.3dshapes/Pin_Header_Angled_2x40_Pitch2.54mm.wrl
-      (at (xyz 0 0 0))
-      (scale (xyz 1 1 1))
-      (rotate (xyz 0 0 0))
-    )
   )
   (module Capacitors_SMD:C_0805 (layer F.Cu)
@@
   (segment (start 228.6 127) (end 231.14 127) (width 0.25) (layer B.Cu) (net 16) (status 80030))
   (segment (start 177.8 127) (end 180.34 127) (width 0.25) (layer B.Cu) (net 16) (status 80030))
-  (segment (start 60.96 114.3) (end 60.96 111.125) (width 0.25) (layer B.Cu) (net 17) (status 400000))
-  (segment (start 149.098 119.38) (end 152.4 119.38) (width 0.25) (layer B.Cu) (net 17) (status 800000))
+  (segment (start 60.96 114.3) (end 60.96 111.125) (width 0.25) (layer B.Cu) (net 17))
+  (segment (start 149.098 119.38) (end 152.4 119.38) (width 0.25) (layer B.Cu) (net 17))
   (segment (start 147.955 118.237) (end 149.098 119.38) (width 0.25) (layer B.Cu) (net 17))
   (segment (start 147.955 110.617) (end 147.955 118.237) (width 0.25) (layer B.Cu) (net 17))
@@
         (xy 63.5 31.496) (xy 76.2 31.496) (xy 80.772 26.924) (xy 86.868 26.924) (xy 91.44 31.496)
         (xy 103.632 31.496) (xy 108.204 26.924) (xy 115.824 26.924) (xy 138.684 49.784) (xy 271.78 49.784)
-        (xy 271.78 56.896) (xy 136.144 56.896) (xy 113.792 34.544) (xy 48.768 34.544) (xy 46.736 36.576)
-        (xy 46.736 39.624) (xy 32.512 53.848) (xy 22.86 53.848) (xy 22.86 48.768) (xy 32.004 48.768)
-        (xy 42.672 38.1) (xy 42.672 35.052) (xy 46.228 31.496) (xy 48.26 31.496) (xy 52.832 26.924)
-        (xy 58.928 26.924)
+        (xy 271.78 56.896) (xy 22.86 56.896) (xy 22.86 48.768) (xy 31.75 48.768) (xy 45.085 35.433)
+        (xy 52.832 26.924) (xy 58.928 26.924)
       )
     )
