File: Spojko_Hardware/Spojko/_saved_SpojkoKonektori.sch (KiCad schematic (older format))
At the start: 22 parts, among them J10 Conn_02x20, J11 Conn_02x14, J20 Conn_02x20, J21 Conn_02x14, J30 Conn_02x20, J31 Conn_02x14, J40 Conn_02x20, J41 Conn_02x14, J50 Conn_02x20, J51 Conn_02x14, J60 Conn_02x20, J61 Conn_02x14, J70 Conn_02x20, J71 Conn_02x14

Commit message: Pre Develope
Connections:
- net GND: now also J10.25 (Pin_25), J10.26 (Pin_26), J10.31 (Pin_31), J10.32 (Pin_32), J10.35 (Pin_35), J10.36 (Pin_36); no longer J10.27 (Pin_27), J10.28 (Pin_28), J10.33 (Pin_33), J10.34 (Pin_34)
- net RST: no longer J10.19 (Pin_19), J10.20 (Pin_20)
- net RXD: now also J10.23 (Pin_23), J10.24 (Pin_24); no longer J10.25 (Pin_25), J10.26 (Pin_26)
- net SCL1: now also J10.27 (Pin_27), J10.28 (Pin_28); no longer J10.29 (Pin_29), J10.30 (Pin_30)
- net SDA: now also J10.33 (Pin_33), J10.34 (Pin_34); no longer J10.35 (Pin_35), J10.36 (Pin_36)
- net SDA1: now also J10.29 (Pin_29), J10.30 (Pin_30); no longer J10.31 (Pin_31), J10.32 (Pin_32)
- net TXD: now also J10.19 (Pin_19), J10.20 (Pin_20); no longer J10.23 (Pin_23), J10.24 (Pin_24)
- new net: J70.17 (Pin_17), J70.18 (Pin_18)
- new net: J70.19 (Pin_19), J70.20 (Pin_20)
- new net: J70.21 (Pin_21), J70.22 (Pin_22)
- new net: J70.23 (Pin_23), J70.24 (Pin_24)
- new net: J70.25 (Pin_25), J70.26 (Pin_26)
- new net: J70.27 (Pin_27), J70.28 (Pin_28)
- new net: J70.29 (Pin_29), J70.30 (Pin_30)
- new net: J70.31 (Pin_31), J70.32 (Pin_32)
- new net: J70.33 (Pin_33), J70.34 (Pin_34)
- new net: J70.35 (Pin_35), J70.36 (Pin_36)
- new net: J70.37 (Pin_37), J70.38 (Pin_38)
- new net: J70.39 (Pin_39), J70.40 (Pin_40)
- new net: J30.17 (Pin_17), J30.18 (Pin_18)
- new net: J30.19 (Pin_19), J30.20 (Pin_20)
- new net: J30.21 (Pin_21), J30.22 (Pin_22)
- new net: J30.39 (Pin_39), J30.40 (Pin_40)
- new net: J40.17 (Pin_17), J40.18 (Pin_18)
- new net: J40.19 (Pin_19), J40.20 (Pin_20)
- new net: J40.21 (Pin_21), J40.22 (Pin_22)
- new net: J40.23 (Pin_23), J40.24 (Pin_24)
- new net: J40.25 (Pin_25), J40.26 (Pin_26)
- new net: J40.27 (Pin_27), J40.28 (Pin_28)
- new net: J40.29 (Pin_29), J40.30 (Pin_30)
- new net: J40.31 (Pin_31), J40.32 (Pin_32)
- new net: J40.33 (Pin_33), J40.34 (Pin_34)
- new net: J40.35 (Pin_35), J40.36 (Pin_36)
- new net: J40.37 (Pin_37), J40.38 (Pin_38)
- new net: J40.39 (Pin_39), J40.40 (Pin_40)
- new net: J50.17 (Pin_17), J50.18 (Pin_18)
- new net: J50.19 (Pin_19), J50.20 (Pin_20)
- new net: J50.21 (Pin_21), J50.22 (Pin_22)
- new net: J50.23 (Pin_23), J50.24 (Pin_24)
- new net: J50.25 (Pin_25), J50.26 (Pin_26)
- new net: J50.27 (Pin_27), J50.28 (Pin_28)
- new net: J50.29 (Pin_29), J50.30 (Pin_30)
- new net: J50.31 (Pin_31), J50.32 (Pin_32)
- new net: J50.33 (Pin_33), J50.34 (Pin_34)
- new net: J50.35 (Pin_35), J50.36 (Pin_36)
- new net: J50.37 (Pin_37), J50.38 (Pin_38)
- new net: J50.39 (Pin_39), J50.40 (Pin_40)
- new net: J60.17 (Pin_17), J60.18 (Pin_18)
- new net: J60.19 (Pin_19), J60.20 (Pin_20)
- new net: J60.21 (Pin_21), J60.22 (Pin_22)
- new net: J60.23 (Pin_23), J60.24 (Pin_24)
- new net: J60.25 (Pin_25), J60.26 (Pin_26)
- new net: J60.27 (Pin_27), J60.28 (Pin_28)
- new net: J60.29 (Pin_29), J60.30 (Pin_30)
- new net: J60.31 (Pin_31), J60.32 (Pin_32)
- new net: J60.33 (Pin_33), J60.34 (Pin_34)
- new net: J60.35 (Pin_35), J60.36 (Pin_36)
- new net: J60.37 (Pin_37), J60.38 (Pin_38)
- new net: J60.39 (Pin_39), J60.40 (Pin_40)
- now unconnected: J20.17 (Pin_17), J20.18 (Pin_18), J20.19 (Pin_19), J20.20 (Pin_20), J20.21 (Pin_21), J20.22 (Pin_22), J20.23 (Pin_23), J20.24 (Pin_24), J20.25 (Pin_25), J20.26 (Pin_26), J20.27 (Pin_27), J20.28 (Pin_28), J20.29 (Pin_29), J20.30 (Pin_30), J20.31 (Pin_31), J20.32 (Pin_32), J20.33 (Pin_33), J20.34 (Pin_34), J20.35 (Pin_35), J20.36 (Pin_36), J20.37 (Pin_37), J20.38 (Pin_38), J20.39 (Pin_39), J20.40 (Pin_40), J30.23 (Pin_23), J30.24 (Pin_24), J30.25 (Pin_25), J30.26 (Pin_26), J30.27 (Pin_27), J30.28 (Pin_28), J30.29 (Pin_29), J30.30 (Pin_30), J30.31 (Pin_31), J30.32 (Pin_32), J30.33 (Pin_33), J30.34 (Pin_34), J30.35 (Pin_35), J30.36 (Pin_36), J30.37 (Pin_37), J30.38 (Pin_38)
