File: Spojko_Hardware/MAX31865_4kanala/MAX31865_4kanala.sch (KiCad schematic (older format))
At the start: 42 parts, among them J1 CONN_01X04, J10 CONN_01X04, J11 CONN_01X04, J12 CONN_01X04, J13 CONN_01X04, J2 CONN_01X04, J3 CONN_01X04, J4 CONN_01X04, J5 CONN_01X40, U1 MAX31865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

Commit message: Ponovno rutovanje i izbacivanje konektora...
Parts:
- removed C13: 4.7uF 25V, Capacitors_SMD:C_1206, symbol C
- removed J10, J11, J12, J13: CONN_01X04, Pin_Headers:Pin_Header_Straight_1x04_Pitch2.54mm, symbol CONN_01X04
Changed lines of the file:
@@
 Wire Wire Line
 	10100 5450 10650 5450
-$Comp
-L CONN_01X04 J10
-U 1 1 5997B427
-P 900 2000
-F 0 "J10" H 900 2250 50  0000 C CNN
-F 1 "CONN_01X04" V 1000 2000 50  0000 C CNN
-F 2 "Pin_Headers:Pin_Header_Straight_1x04_Pitch2.54mm" H 900 2000 50  0001 C CNN
-F 3 "" H 900 2000 50  0001 C CNN
-	1    900  2000
-	-1   0    0    1
-$EndComp
-Text Label 1650 1850 2    60   ~ 0
-FORCE0-
-Text Label 1650 1950 2    60   ~ 0
-RTDIN0-
-Text Label 1650 2050 2    60   ~ 0
-RTDIN0+
-Text Label 1650 2150 2    60   ~ 0
-IFORCE0+
-Wire Wire Line
-	1650 1850 1100 1850
-Wire Wire Line
-	1100 1950 1650 1950
-Wire Wire Line
-	1650 2050 1100 2050
-Wire Wire Line
-	1100 2150 1650 2150
-$Comp
-L CONN_01X04 J11
-U 1 1 5997C85A
-P 900 3700
-F 0 "J11" H 900 3950 50  0000 C CNN
-F 1 "CONN_01X04" V 1000 3700 50  0000 C CNN
-F 2 "Pin_Headers:Pin_Header_Straight_1x04_Pitch2.54mm" H 900 3700 50  0001 C CNN
-F 3 "" H 900 3700 50  0001 C CNN
-	1    900  3700
-	-1   0    0    1
-$EndComp
-Text Label 1650 3550 2    60   ~ 0
-FORCE1-
-Text Label 1650 3650 2    60   ~ 0
-RTDIN1-
-Text Label 1650 3750 2    60   ~ 0
-RTDIN1+
-Text Label 1650 3850 2    60   ~ 0
-IFORCE1+
-Wire Wire Line
-	1650 3550 1100 3550
-Wire Wire Line
-	1100 3650 1650 3650
-Wire Wire Line
-	1650 3750 1100 3750
-Wire Wire Line
-	1100 3850 1650 3850
-$Comp
-L CONN_01X04 J12
-U 1 1 5997C903
-P 900 5400
-F 0 "J12" H 900 5650 50  0000 C CNN
-F 1 "CONN_01X04" V 1000 5400 50  0000 C CNN
-F 2 "Pin_Headers:Pin_Header_Straight_1x04_Pitch2.54mm" H 900 5400 50  0001 C CNN
-F 3 "" H 900 5400 50  0001 C CNN
-	1    900  5400
-	-1   0    0    1
-$EndComp
-Text Label 1650 5250 2    60   ~ 0
-FORCE2-
-Text Label 1650 5350 2    60   ~ 0
-RTDIN2-
-Text Label 1650 5450 2    60   ~ 0
-RTDIN2+
-Text Label 1650 5550 2    60   ~ 0
-IFORCE2+
-Wire Wire Line
-	1650 5250 1100 5250
-Wire Wire Line
-	1100 5350 1650 5350
-Wire Wire Line
-	1650 5450 1100 5450
-Wire Wire Line
-	1100 5550 1650 5550
-$Comp
-L CONN_01X04 J13
-U 1 1 5997C9E3
-P 900 7100
-F 0 "J13" H 900 7350 50  0000 C CNN
-F 1 "CONN_01X04" V 1000 7100 50  0000 C CNN
-F 2 "Pin_Headers:Pin_Header_Straight_1x04_Pitch2.54mm" H 900 7100 50  0001 C CNN
-F 3 "" H 900 7100 50  0001 C CNN
-	1    900  7100
-	-1   0    0    1
-$EndComp
-Text Label 1650 6950 2    60   ~ 0
-FORCE3-
-Text Label 1650 7050 2    60   ~ 0
-RTDIN3-
-Text Label 1650 7150 2    60   ~ 0
-RTDIN3+
-Text Label 1650 7250 2    60   ~ 0
-IFORCE3+
-Wire Wire Line
-	1650 6950 1100 6950
-Wire Wire Line
-	1100 7050 1650 7050
-Wire Wire Line
-	1650 7150 1100 7150
-Wire Wire Line
-	1100 7250 1650 7250
-$Comp
-L C C13
-U 1 1 5997ECE6
-P 10200 3500
-F 0 "C13" H 10225 3600 50  0000 L CNN
-F 1 "4.7uF 25V" H 10225 3400 50  0000 L CNN
-F 2 "Capacitors_SMD:C_1206" H 10238 3350 50  0001 C CNN
-F 3 "" H 10200 3500 50  0001 C CNN
-	1    10200 3500
-	1    0    0    -1
-$EndComp
-Wire Wire Line
-	10200 3350 10200 3250
-Connection ~ 10200 3250
-Wire Wire Line
-	10200 3650 10200 3750
-Wire Wire Line
-	10200 3750 10450 3750
-Connection ~ 10450 3750
 Wire Wire Line
 	10450 3050 10450 6300

Commit message: Izmene predlozi matori
Parts:
- removed J1, J2, J3, J4: CONN_01X04, Socket_Strips:Socket_Strip_Straight_1x04_Pitch2.54mm, symbol CONN_01X04
- added J1, J2, J3, J4: 1824763, 1824763, symbol 1824763
Connections:
- net FORCE0-: now also J1.3
- net FORCE1-: now also J2.3
- net FORCE2-: now also J3.3
- net FORCE3-: now also J4.3
- net IFORCE0+: now also J1.1
- net IFORCE1+: now also J2.1
- net IFORCE2+: now also J3.1
- net IFORCE3+: now also J4.1
- net RTDIN0+: now also J1.2
- net RTDIN0-: now also J1.4
- net RTDIN1+: now also J2.2
- net RTDIN1-: now also J2.4
- net RTDIN2+: now also J3.2
- net RTDIN2-: now also J3.4
- net RTDIN3+: now also J4.2
- net RTDIN3-: now also J4.4

Commit message: Added gif main ReadMe
Parts:
- removed C11, C12, C7, C8: C, Capacitors_SMD:C_0805, symbol C
- removed C3, C4: 0.1uF 25V, X7R, Capacitors_SMD:C_0805, symbol C
- removed J1, J2, J3, J4: 1824763, 1824763, symbol 1824763
- removed R10, R6, R7, R9: 150, Resistors_SMD:R_0805, symbol R
- removed R3, R4: 400, Resistors_SMD:R_0805, symbol R
- removed U3, U4: MAX31865, project_footprints:QFN-20-1EP_5x5mm_Pitch0.65mm, symbol MAX31865
- added J1, J2: CONN_01X04, Connectors_Phoenix:PhoenixContact_MC-GF_04x3.81mm_Angled_ThreadedFlange_MountHole, symbol CONN_01X04
- added R? (x2): R, symbol R
- added U? (x2): PC817, Housings_DIP:DIP-4_W7.62mm, symbol PC817
Connections:
- net FORCE0-: now also J1.4 (P4)
- net FORCE1-: now also J2.4 (P4)
- net GND: now also U5.23 (GND), U5.29 (GND2), U5.4 (GND1), U?.2, U?.2
- net IFORCE0+: now also J1.1 (P1)
- net IFORCE1+: now also J2.1 (P1)
- net RTDIN0+: now also J1.2 (P2)
- net RTDIN0-: now also J1.3 (P3)
- net RTDIN1+: now also J2.2 (P2)
- net RTDIN1-: now also J2.3 (P3)
- net DO1: now reaches U5.9 (D6)
- net DO1: now also R?.1
- net CS2: no longer names the net of U5.7 (D4)
- net CS3 renamed DO0
- net DO0: now also R?.1
- new net: R?.2, U?.1 (x2)
