File: Kontroler_Hardware/New folder/New folder.sch (KiCad schematic (older format))
At the start: 1 part

Commit message: Dodao kondenzator
Parts:
- added C? (x2): C, symbol device:C
- added R?: 10K, symbol device:R
Connections:
- net labels removed: V5
- wire segments 3 -> 5
Changed lines of the file:
@@
 Wire Wire Line
 	3050 2200 3050 1950
-Text GLabel 4400 1950 2    50   Input ~ 0
-V5
 Text GLabel 4400 3600 2    50   Input ~ 0
 GND
 Wire Wire Line
 	4400 3600 3050 3600
+$Comp
+L device:R R?
+U 1 1 5ADDDE04
+P 5150 1950
+F 0 "R?" V 5357 1950 50  0000 C CNN
+F 1 "10K" V 5266 1950 50  0000 C CNN
+F 2 "" V 5080 1950 50  0001 C CNN
+F 3 "" H 5150 1950 50  0001 C CNN
+	1    5150 1950
+	0    -1   -1   0
+$EndComp
 Wire Wire Line
-	3050 1950 4400 1950
+	3050 1950 5000 1950
+$Comp
+L device:C C?
+U 1 1 5ADDDFA8
+P 5500 2350
+F 0 "C?" H 5615 2396 50  0000 L CNN
+F 1 "C" H 5615 2305 50  0000 L CNN
+F 2 "" H 5538 2200 50  0001 C CNN
+F 3 "" H 5500 2350 50  0001 C CNN
+	1    5500 2350
+	1    0    0    -1
+$EndComp
+Wire Wire Line
+	5300 1950 5500 1950
+Wire Wire Line
+	5500 1950 5500 2200
+$Comp
+L device:C C?
+U 1 1 5ADDE06B
+P 6600 2850
+F 0 "C?" H 6715 2896 50  0000 L CNN
+F 1 "C" H 6715 2805 50  0000 L CNN
+F 2 "" H 6638 2700 50  0001 C CNN
+F 3 "" H 6600 2850 50  0001 C CNN
+	1    6600 2850
+	1    0    0    -1
+$EndComp
 $EndSCHEMATC
