File: Kontroler_Hardware/Spojko/Napajanje_3V3.sch (KiCad schematic (older format))
At the start: 1 part, among them U5 vLM2596

Commit message: Puno izmena
Parts:
- added C102: CP, Capacitors_THT:CP_Radial_D12.5mm_P7.50mm, symbol Spojko-rescue:CP
- U5: symbol vLM2596 -> Spojko-rescue:vLM2596
Connections:
- net GND24V: now also C102.2
- net In_24V: now also C102.1
Changed lines of the file:
@@
-EESchema Schematic File Version 2
+EESchema Schematic File Version 4
 LIBS:Spojko-cache
-LIBS:power
-LIBS:device
-LIBS:transistors
-LIBS:conn
-LIBS:linear
-LIBS:regul
-LIBS:74xx
-LIBS:cmos4000
-LIBS:adc-dac
-LIBS:memory
-LIBS:xilinx
-LIBS:microcontrollers
-LIBS:dsp
-LIBS:microchip
-LIBS:analog_switches
-LIBS:motorola
-LIBS:texas
-LIBS:intel
-LIBS:audio
-LIBS:interface
-LIBS:digital-audio
-LIBS:philips
-LIBS:display
-LIBS:cypress
-LIBS:siliconi
-LIBS:opto
-LIBS:atmel
-LIBS:contrib
-LIBS:valves
-LIBS:Symbols_DCDC-ACDC-Converter_RevC_20Jul2012
-LIBS:Symbols_EN60617_13Mar2013
-LIBS:Symbols_EN60617-10_HF-Radio_DRAFT_12Sep2013
-LIBS:Symbols_ICs-Diskrete_RevD10
-LIBS:Symbols_ICs-Opto_RevB_16Sep2013
-LIBS:Symbols_Microcontroller_Philips-NXP_RevA_06Oct2013
-LIBS:Symbols_Socket-DIN41612_RevA
-LIBS:Symbols_Transformer-Diskrete_RevA
-LIBS:SymbolsSimilarEN60617+oldDIN617-RevE8
-LIBS:switches
-LIBS:sensors
-EELAYER 25 0
+EELAYER 26 0
 EELAYER END
 $Descr A4 11693 8268
 encoding utf-8
-Sheet 5 5
+Sheet 4 5
 Title ""
 Date ""
@@
 Out_3V3
 $Comp
-L GND #PWR05
+L Spojko-rescue:GND #PWR05
 U 1 1 5985541E
 P 7950 4000
@@
 $EndComp
 Wire Wire Line
-	3500 4000 4500 4000
-Wire Wire Line
 	6900 4000 7950 4000
-Wire Wire Line
-	4500 3700 3500 3700
 $Comp
-L vLM2596 U5
+L Spojko-rescue:vLM2596 U5
 U 1 1 5985A430
 P 5750 3850
@@
 Wire Wire Line
 	6900 3700 8000 3700
+$Comp
+L Spojko-rescue:CP C102
+U 1 1 5AD95880
+P 4100 3850
+F 0 "C102" H 4125 3950 50  0000 L CNN
+F 1 "CP" H 4125 3750 50  0000 L CNN
+F 2 "Capacitors_THT:CP_Radial_D12.5mm_P7.50mm" H 4138 3700 50  0001 C CNN
+F 3 "" H 4100 3850 50  0001 C CNN
+	1    4100 3850
+	1    0    0    -1
+$EndComp
+Wire Wire Line
+	3500 3700 4500 3700
+Connection ~ 4100 3700
+Wire Wire Line
+	3500 4000 4500 4000
+Connection ~ 4100 4000
 $EndSCHEMATC

Commit message: NewTemplates
Parts:
- U5: footprint project_footprints:Napajanje_5V -> lib_fp:Napajanje_5V
Changed lines of the file:
@@
 F 0 "U5" H 4800 4150 60  0000 C CNN
 F 1 "vLM2596" H 4900 3550 60  0000 C CNN
-F 2 "project_footprints:Napajanje_5V" H 5750 3850 60  0001 C CNN
+F 2 "lib_fp:Napajanje_5V" H 5750 3850 60  0001 C CNN
 F 3 "" H 5750 3850 60  0001 C CNN
 	1    5750 3850
@@
 $EndComp
 Wire Wire Line
-	3500 3700 4500 3700
+	3500 3700 4100 3700
 Connection ~ 4100 3700
 Wire Wire Line
-	3500 4000 4500 4000
+	3500 4000 4100 4000
 Connection ~ 4100 4000
+Wire Wire Line
+	4100 3700 4500 3700
+Wire Wire Line
+	4100 4000 4500 4000
 $EndSCHEMATC
