File: Kontroler_Hardware/Spojko/PowerSupply5V.sch (KiCad schematic (older format))
At the start: 1 part, among them U3 vLM2596

Commit message: Puno izmena
Parts:
- added C100: CP, Capacitors_THT:CP_Radial_D12.5mm_P7.50mm, symbol Spojko-rescue:CP
- U3: symbol vLM2596 -> Spojko-rescue:vLM2596
Connections:
- net 24V_In: now also C100.1
- net GND24V: now also C100.2
Changed lines of the file:
@@
-EESchema Schematic File Version 2
+EESchema Schematic File Version 4
 LIBS:Spojko-cache
-LIBS:power
-LIBS:device
-LIBS:transistors
-LIBS:conn
-LIBS:linear
-LIBS:regul
-LIBS:74xx
-LIBS:cmos4000
-LIBS:adc-dac
-LIBS:memory
-LIBS:xilinx
-LIBS:microcontrollers
-LIBS:dsp
-LIBS:microchip
-LIBS:analog_switches
-LIBS:motorola
-LIBS:texas
-LIBS:intel
-LIBS:audio
-LIBS:interface
-LIBS:digital-audio
-LIBS:philips
-LIBS:display
-LIBS:cypress
-LIBS:siliconi
-LIBS:opto
-LIBS:atmel
-LIBS:contrib
-LIBS:valves
-LIBS:Symbols_DCDC-ACDC-Converter_RevC_20Jul2012
-LIBS:Symbols_EN60617_13Mar2013
-LIBS:Symbols_EN60617-10_HF-Radio_DRAFT_12Sep2013
-LIBS:Symbols_ICs-Diskrete_RevD10
-LIBS:Symbols_ICs-Opto_RevB_16Sep2013
-LIBS:Symbols_Microcontroller_Philips-NXP_RevA_06Oct2013
-LIBS:Symbols_Socket-DIN41612_RevA
-LIBS:Symbols_Transformer-Diskrete_RevA
-LIBS:SymbolsSimilarEN60617+oldDIN617-RevE8
-LIBS:switches
-LIBS:sensors
-EELAYER 25 0
+EELAYER 26 0
 EELAYER END
 $Descr A4 11693 8268
 encoding utf-8
-Sheet 3 5
+Sheet 2 5
 Title ""
 Date ""
@@
 $EndDescr
 $Comp
-L vLM2596 U3
+L Spojko-rescue:vLM2596 U3
 U 1 1 597BCF43
 P 5850 3900
@@
 Wire Wire Line
 	7000 4050 8000 4050
-Wire Wire Line
-	3500 4050 4600 4050
-Wire Wire Line
-	3500 3750 4600 3750
 Text Notes 5300 3950 0    60   ~ 0
 Kartica Napajanja 5V
@@
 GND24V
 $Comp
-L GND #PWR03
+L Spojko-rescue:GND #PWR03
 U 1 1 597BD727
 P 8000 4050
@@
 	1    0    0    -1
 $EndComp
+$Comp
+L Spojko-rescue:CP C100
+U 1 1 5AD9516F
+P 4300 3900
+F 0 "C100" H 4325 4000 50  0000 L CNN
+F 1 "CP" H 4325 3800 50  0000 L CNN
+F 2 "Capacitors_THT:CP_Radial_D12.5mm_P7.50mm" H 4338 3750 50  0001 C CNN
+F 3 "" H 4300 3900 50  0001 C CNN
+	1    4300 3900
+	1    0    0    -1
+$EndComp
+Wire Wire Line
+	3500 3750 4600 3750
+Connection ~ 4300 3750
+Wire Wire Line
+	3500 4050 4600 4050
+Connection ~ 4300 4050
 $EndSCHEMATC

Commit message: NewTemplates
Parts:
- added C? (x2): CP, Capacitors_THT:CP_Radial_D12.5mm_P7.50mm, symbol Spojko-rescue:CP
- added U? (x2): vLM2596, lib_fp:Napajanje_5V, symbol Spojko-rescue:vLM2596
- U3: footprint project_footprints:Napajanje_5V -> lib_fp:Napajanje_5V
Connections:
- net GND: now also U?.3 (GND), U?.3 (GND)
- net GND24V: now also C?.2, C?.2, U?.1 (GND), U?.1 (GND)
- net 24V_In renamed In_24V
- net In_24V: now also C?.1, C?.1, U?.2 (24V_In), U?.2 (24V_In)
- net 5V_Out renamed Out5VMCU
- new net Out5V: U?.4 (5V_Out)
- new net Out_3V3: U?.4 (5V_Out)
Other:
- moved on the sheet: C100, U3
Changed lines of the file:
@@
 $Descr A4 11693 8268
 encoding utf-8
-Sheet 2 5
+Sheet 2 3
 Title ""
 Date ""
@@
 L Spojko-rescue:vLM2596 U3
 U 1 1 597BCF43
-P 5850 3900
-F 0 "U3" H 4900 4200 60  0000 C CNN
-F 1 "vLM2596" H 5000 3550 60  0000 C CNN
-F 2 "project_footprints:Napajanje_5V" H 5850 3900 60  0001 C CNN
-F 3 "" H 5850 3900 60  0001 C CNN
-	1    5850 3900
+P 5450 1600
+F 0 "U3" H 4500 1900 60  0000 C CNN
+F 1 "vLM2596" H 4600 1250 60  0000 C CNN
+F 2 "lib_fp:Napajanje_5V" H 5450 1600 60  0001 C CNN
+F 3 "" H 5450 1600 60  0001 C CNN
+	1    5450 1600
 	1    0    0    -1
 $EndComp
 Wire Wire Line
-	7000 4050 8000 4050
-Text Notes 5300 3950 0    60   ~ 0
+	6600 1750 7600 1750
+Text Notes 4900 1650 0    60   ~ 0
 Kartica Napajanja 5V
-Text HLabel 3500 3750 0    60   Input ~ 0
-24V_In
-Text HLabel 7950 3750 2    60   Input ~ 0
-5V_Out
+Text HLabel 7550 1450 2    60   Input ~ 0
+Out5VMCU
 Wire Wire Line
-	7000 3750 7950 3750
-Text GLabel 3500 4050 0    60   Input ~ 0
+	6600 1450 7550 1450
+Text GLabel 3100 1750 0    60   Input ~ 0
 GND24V
 $Comp
 L Spojko-rescue:GND #PWR03
 U 1 1 597BD727
-P 8000 4050
-F 0 "#PWR03" H 8000 3800 50  0001 C CNN
-F 1 "GND" H 8000 3900 50  0000 C CNN
-F 2 "" H 8000 4050 50  0001 C CNN
-F 3 "" H 8000 4050 50  0001 C CNN
-	1    8000 4050
+P 7600 1750
+F 0 "#PWR03" H 7600 1500 50  0001 C CNN
+F 1 "GND" H 7600 1600 50  0000 C CNN
+F 2 "" H 7600 1750 50  0001 C CNN
+F 3 "" H 7600 1750 50  0001 C CNN
+	1    7600 1750
 	1    0    0    -1
 $EndComp
@@
 L Spojko-rescue:CP C100
 U 1 1 5AD9516F
-P 4300 3900
-F 0 "C100" H 4325 4000 50  0000 L CNN
-F 1 "CP" H 4325 3800 50  0000 L CNN
-F 2 "Capacitors_THT:CP_Radial_D12.5mm_P7.50mm" H 4338 3750 50  0001 C CNN
-F 3 "" H 4300 3900 50  0001 C CNN
-	1    4300 3900
+P 3900 1600
+F 0 "C100" H 3925 1700 50  0000 L CNN
+F 1 "CP" H 3925 1500 50  0000 L CNN
+F 2 "Capacitors_THT:CP_Radial_D12.5mm_P7.50mm" H 3938 1450 50  0001 C CNN
+F 3 "" H 3900 1600 50  0001 C CNN
+	1    3900 1600
+	1    0    0    -1
+$EndComp
+Connection ~ 3900 1450
+Wire Wire Line
+	3100 1750 3900 1750
+Connection ~ 3900 1750
+Wire Wire Line
+	3900 1450 4200 1450
+Wire Wire Line
+	3900 1750 4200 1750
+$Comp
+L Spojko-rescue:vLM2596 U?
+U 1 1 5AEC32C0
+P 5350 3750
+F 0 "U?" H 4400 4050 60  0000 C CNN
+F 1 "vLM2596" H 4500 3400 60  0000 C CNN
+F 2 "lib_fp:Napajanje_5V" H 5350 3750 60  0001 C CNN
+F 3 "" H 5350 3750 60  0001 C CNN
+	1    5350 3750
+	1    0    0    -1
+$EndComp
+$Comp
+L Spojko-rescue:GND #PWR?
+U 1 1 5AEC32C7
+P 7400 3900
+F 0 "#PWR?" H 7400 3650 50  0001 C CNN
+F 1 "GND" H 7400 3750 50  0000 C CNN
+F 2 "" H 7400 3900 50  0001 C CNN
+F 3 "" H 7400 3900 50  0001 C CNN
+	1    7400 3900
+	1    0    0    -1
+$EndComp
+Text HLabel 7400 3600 2    60   Input ~ 0
+Out5V
+Text GLabel 3300 3900 0    60   Input ~ 0
+GND24V
+Wire Wire Line
+	6500 3900 7400 3900
+Wire Wire Line
+	6500 3600 7400 3600
+$Comp
+L Spojko-rescue:CP C?
+U 1 1 5AEC32D2
+P 3800 3750
+F 0 "C?" H 3825 3850 50  0000 L CNN
+F 1 "CP" H 3825 3650 50  0000 L CNN
+F 2 "Capacitors_THT:CP_Radial_D12.5mm_P7.50mm" H 3838 3600 50  0001 C CNN
+F 3 "" H 3800 3750 50  0001 C CNN
+	1    3800 3750
+	1    0    0    -1
+$EndComp
+Connection ~ 3800 3600
+Wire Wire Line
+	3300 3900 3800 3900
+Connection ~ 3800 3900
+Wire Wire Line
+	3800 3600 4100 3600
+Wire Wire Line
+	3800 3900 4100 3900
+Text HLabel 7700 4950 2    60   Input ~ 0
+Out_3V3
+$Comp
+L Spojko-rescue:GND #PWR?
+U 1 1 5AEC35AB
+P 7650 5250
+F 0 "#PWR?" H 7650 5000 50  0001 C CNN
+F 1 "GND" H 7650 5100 50  0000 C CNN
+F 2 "" H 7650 5250 50  0001 C CNN
+F 3 "" H 7650 5250 50  0001 C CNN
+	1    7650 5250
+	0    -1   -1   0
+$EndComp
+Wire Wire Line
+	6600 5250 7650 5250
+$Comp
+L Spojko-rescue:vLM2596 U?
+U 1 1 5AEC35B2
+P 5450 5100
+F 0 "U?" H 4500 5400 60  0000 C CNN
+F 1 "vLM2596" H 4600 4800 60  0000 C CNN
+F 2 "lib_fp:Napajanje_5V" H 5450 5100 60  0001 C CNN
+F 3 "" H 5450 5100 60  0001 C CNN
+	1    5450 5100
+	1    0    0    -1
+$EndComp
+Text GLabel 3200 5250 0    60   Input ~ 0
+GND24V
+Wire Wire Line
+	6600 4950 7700 4950
+$Comp
+L Spojko-rescue:CP C?
+U 1 1 5AEC35BB
+P 3800 5100
+F 0 "C?" H 3825 5200 50  0000 L CNN
+F 1 "CP" H 3825 5000 50  0000 L CNN
+F 2 "Capacitors_THT:CP_Radial_D12.5mm_P7.50mm" H 3838 4950 50  0001 C CNN
+F 3 "" H 3800 5100 50  0001 C CNN
+	1    3800 5100
 	1    0    0    -1
 $EndComp
 Wire Wire Line
-	3500 3750 4600 3750
-Connection ~ 4300 3750
+	3200 4950 3800 4950
+Connection ~ 3800 4950
 Wire Wire Line
-	3500 4050 4600 4050
-Connection ~ 4300 4050
+	3200 5250 3800 5250
+Connection ~ 3800 5250
+Wire Wire Line
+	3800 4950 4200 4950
+Wire Wire Line
+	3800 5250 4200 5250
+Text Notes 4850 3800 0    60   ~ 0
+Kartica Napajanja 5V
+Text Notes 4900 5200 0    60   ~ 0
+Kartica Napajanja 5V
+Wire Wire Line
+	3300 3600 3800 3600
+Wire Wire Line
+	3100 1450 3900 1450
+Text HLabel 3200 4950 0    60   Input ~ 0
+In_24V
+Text HLabel 3300 3600 0    60   Input ~ 0
+In_24V
+Text HLabel 3100 1450 0    60   Input ~ 0
+In_24V
 $EndSCHEMATC
