File: Kontroler_Hardware/Spojko/Spojko.kicad_pcb (KiCad board)
At the start: 2 copper layers, 254 x 139.7 mm, 42 parts, among them J1 CONN_01X02, J2 CONN_01X06, J3 CONN_02X40, J4 CONN_02X40, J5 CONN_02X40, J6 CONN_02X40, J7 CONN_02X40, J8 CONN_02X40, P1 Raspberry_Pi, Q1 BSS138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

Commit message: Puno izmena
Parts:
- added C100: CP, Capacitors_THT:CP_Radial_D12.5mm_P7.50mm, F.Cu at (46.2, 25.2)
- added C101: CP, Capacitors_THT:CP_Radial_D12.5mm_P7.50mm, F.Cu at (72.1, 6.87)
- added C102: CP, Capacitors_THT:CP_Radial_D12.5mm_P7.50mm, F.Cu at (108.2, 2.30)
- J1: footprint Connectors:bornier2 -> Connectors_Phoenix:PhoenixContact_GMSTBA-G_02x7.62mm_Angled
- moved U3 9.42 mm to (57.9, 37.3)
- moved C1 4.08 mm to (46.7, 79.0)
- moved C4 4.08 mm to (102.6, 79.0)
- moved C7 4.08 mm to (74.7, 79.0)
- moved J1 0.37 mm to (26.4, 45.5)

Commit message: Deleted  PCB Spojko
Parts:
- removed C1, C4, C7: CP, Capacitors_SMD:CP_Elec_8x6.7
- removed C100, C101, C102: CP, Capacitors_THT:CP_Radial_D12.5mm_P7.50mm
- removed C2, C5: C, Capacitors_SMD:C_0805
- removed C3, C6: C, Capacitors_Tantalum_SMD:CP_Tantalum_Case-A_EIA-3216-18_Reflow
- removed J1: CONN_01X02, Connectors_Phoenix:PhoenixContact_GMSTBA-G_02x7.62mm_Angled
- removed J2: CONN_01X06, Pin_Headers:Pin_Header_Straight_1x06_Pitch2.54mm
- removed J3, J4, J5, J6, J7: CONN_02X40, Pin_Headers:Pin_Header_Straight_2x40_Pitch2.54mm
- removed J8: CONN_02X40, Pin_Headers:Pin_Header_Angled_2x40_Pitch2.54mm
- removed JP1, JP10, JP2, JP3, JP4, JP5, JP6, JP7, JP8, JP9: NO, Pin_Headers:Pin_Header_Straight_1x02_Pitch2.54mm
- removed P1: Raspberry_Pi, Pin_Headers:Pin_Header_Straight_2x20_Pitch2.54mm
- removed Q1, Q2: BSS138, TO_SOT_Packages_SMD:SOT-23
- removed R1, R2, R9: 10K, Resistors_SMD:R_1206
- removed R3, R4: 4K7, Resistors_SMD:R_0805
- removed R5, R6: 10K, Resistors_SMD:R_0805
- removed SW1: SW_Reset, Buttons_Switches_SMD:SW_SPST_EVPBF
- removed SW2: SW_Flash, Buttons_Switches_SMD:SW_SPST_EVPBF
- removed U1: ESP-12E, project_footprints:ESP-12E
- removed U3, U4, U5: vLM2596, project_footprints:Napajanje_5V
- removed U6: DHT11, project_footprints:DHT22_Temperature_Humidity
Routing:
- net TXD: track 235.4 -> 0.00 mm, vias 5 -> 0
- net RXD: track 226.9 -> 0.00 mm, vias 4 -> 0
- net SCL: track 225.6 -> 0.00 mm
- net RST: track 225.4 -> 0.00 mm, vias 4 -> 0
- net SDA: track 217.2 -> 0.00 mm
- net SDA1: track 144.1 -> 0.00 mm
- net SCL1: track 139.4 -> 0.00 mm, vias 1 -> 0
- net Net-(J3-Pad41): track 136.5 -> 0.00 mm
- net Net-(J3-Pad37): track 135.5 -> 0.00 mm
- net Net-(J3-Pad35): track 134.9 -> 0.00 mm
- net Net-(J3-Pad33): track 134.4 -> 0.00 mm
- net Net-(J3-Pad31): track 133.9 -> 0.00 mm
- net Net-(J3-Pad27): track 133.9 -> 0.00 mm
- net Net-(J3-Pad29): track 133.4 -> 0.00 mm
- net GPIO20: track 127.3 -> 0.00 mm, vias 2 -> 0
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- removed copper zone on B.Cu, net +24V
- removed copper zone on B.Cu, net +3V3
- removed copper zone on B.Cu, net +5V
- removed copper zone on F.Cu, net GND
- removed copper zone on F.Cu, net GND24V
Other:
- board outline removed

Commit message: NewTemplates
Parts:
- added J10: Conn_02x20, Connector_PinHeader_2.54mm:PinHeader_2x20_P2.54mm_Vertical, F.Cu at (214.6, 91.4)
- added J11: Conn_02x14, Connector_PinHeader_2.54mm:PinHeader_2x14_P2.54mm_Vertical, F.Cu at (214.6, 146.1)
- added J20: Conn_02x20, Connector_PinHeader_2.54mm:PinHeader_2x20_P2.54mm_Vertical, F.Cu at (238.8, 91.4)
- added J21: Conn_02x14, Connector_PinHeader_2.54mm:PinHeader_2x14_P2.54mm_Vertical, F.Cu at (238.8, 146.1)
- added J30: Conn_02x20, Connector_PinHeader_2.54mm:PinHeader_2x20_P2.54mm_Vertical, F.Cu at (264.2, 91.4)
- added J31: Conn_02x14, Connector_PinHeader_2.54mm:PinHeader_2x14_P2.54mm_Vertical, F.Cu at (264.2, 146.1)
- added J40: Conn_02x20, Connector_PinHeader_2.54mm:PinHeader_2x20_P2.54mm_Vertical, F.Cu at (289.6, 91.4)
- added J41: Conn_02x14, Connector_PinHeader_2.54mm:PinHeader_2x14_P2.54mm_Vertical, F.Cu at (289.6, 146.1)
- added J50: Conn_02x20, Connector_PinHeader_2.54mm:PinHeader_2x20_P2.54mm_Vertical, F.Cu at (315.0, 91.4)
- added J51: Conn_02x14, Connector_PinHeader_2.54mm:PinHeader_2x14_P2.54mm_Vertical, F.Cu at (315.0, 146.1)
- added J60: Conn_02x20, Connector_PinHeader_2.54mm:PinHeader_2x20_P2.54mm_Vertical, F.Cu at (340.4, 91.4)
- added J61: Conn_02x14, Connector_PinHeader_2.54mm:PinHeader_2x14_P2.54mm_Vertical, F.Cu at (341.6, 146.1)
- added J70: Conn_02x20, Connector_PinHeader_2.54mm:PinHeader_2x20_P2.54mm_Horizontal, F.Cu at (350.5, 91.4)
- added J71: Conn_02x14, Connector_PinHeader_2.54mm:PinHeader_2x14_P2.54mm_Horizontal, F.Cu at (350.5, 146.1)
- added P1: Raspberry_Pi, Connector_PinHeader_2.54mm:PinHeader_2x20_P2.54mm_Vertical, F.Cu at (110.5, 95.2)
- added Q1: BSS138, Package_TO_SOT_SMD:SOT-23, F.Cu at (164.9, 119.1)
- added Q2: BSS138, Package_TO_SOT_SMD:SOT-23, F.Cu at (181.4, 106.3)
- added R1: 10K, Resistor_SMD:R_1206_3216Metric, F.Cu at (164.2, 126.3)
- added R2: 10K, Resistor_SMD:R_1206_3216Metric, F.Cu at (171.3, 118.5)
- added R5: 10K, Resistor_SMD:R_0805_2012Metric, F.Cu at (180.2, 113.3)
- added U1: ESP-12E, lib_fp:ESP-12E, F.Cu at (144.8, 97.8)
- added U3: vLM2596, lib_fp:Napajanje_5V, F.Cu at (151.1, 179.1)
- added U4: vLM2596, lib_fp:Napajanje_5V, F.Cu at (121.9, 179.1)
- added U5: vLM2596, lib_fp:Napajanje_5V, F.Cu at (179.1, 179.1)
- added U6: DHT11, lib_fp:DHT22_Temperature_Humidity, F.Cu at (193.0, 91.4)
Other:
- board outline added: 300 x 107.3 mm
