File: Kontroler_Hardware/template/SpojkoMainPowerTemplate/SpojkoMainPowerTemplate.kicad_pcb (KiCad board)
At the start: 2 copper layers, 100 x 100 mm, 0 parts

Commit message: Finish templates
Parts:
- added J1: Conn_02x14_Odd_Even, Connector_PinHeader_2.54mm:PinHeader_2x14_P2.54mm_Horizontal, F.Cu at (113.0, 133.3)
